Commit message: Added odom frame in simulation

File: install/taurob_tracker_simulation/taurob_tracker_description/urdf/taurob_tracker_flipper_indoor.xacro (robot description, xacro)
@@ -45,4 +45,10 @@
     <xacro:include filename="$(find hector_sensors_description)/urdf/flir_a35_camera.urdf.xacro"/>
     <link name="base_link"/>
+    <joint name="odom_joint" type="fixed">
+      <origin xyz="${-tracker_base_offset_x} 0 0.193" rpy="0 0 0"/>
+      <parent link="base_link"/>
+      <child link="odom"/>
+    </joint>
+    <link name="odom"/>
     <joint name="chassis_joint" type="fixed">
       <origin xyz="${-tracker_base_offset_x} 0 0.193" rpy="0 0 0"/>

File: install/taurob_tracker_simulation/taurob_tracker_description/urdf/taurob_tracker_flipper_outdoor.xacro (robot description, xacro)
@@ -44,4 +44,9 @@
     <xacro:include filename="$(find hector_sensors_description)/urdf/flir_a35_camera.urdf.xacro"/>
     <link name="base_link"/>
+    <joint name="odom_joint" type="fixed">
+      <origin xyz="${-tracker_base_offset_x} 0 0.193" rpy="0 0 0"/>
+      <parent link="base_link"/>
+      <child link="odom"/>
+    </joint>
     <joint name="chassis_joint" type="fixed">
       <origin xyz="${-tracker_base_offset_x} 0 0.193" rpy="0 0 0"/>

Commit message: Bug fix odom Added gps coordinates for AKW

File: install/taurob_tracker_simulation/taurob_tracker_description/urdf/taurob_tracker_flipper_indoor.xacro (robot description, xacro)
@@ -45,10 +45,4 @@
     <xacro:include filename="$(find hector_sensors_description)/urdf/flir_a35_camera.urdf.xacro"/>
     <link name="base_link"/>
-    <joint name="odom_joint" type="fixed">
-      <origin xyz="${-tracker_base_offset_x} 0 0.193" rpy="0 0 0"/>
-      <parent link="base_link"/>
-      <child link="odom"/>
-    </joint>
-    <link name="odom"/>
     <joint name="chassis_joint" type="fixed">
       <origin xyz="${-tracker_base_offset_x} 0 0.193" rpy="0 0 0"/>

File: install/taurob_tracker_simulation/taurob_tracker_description/urdf/taurob_tracker_flipper_outdoor.xacro (robot description, xacro)
@@ -44,9 +44,4 @@
     <xacro:include filename="$(find hector_sensors_description)/urdf/flir_a35_camera.urdf.xacro"/>
     <link name="base_link"/>
-    <joint name="odom_joint" type="fixed">
-      <origin xyz="${-tracker_base_offset_x} 0 0.193" rpy="0 0 0"/>
-      <parent link="base_link"/>
-      <child link="odom"/>
-    </joint>
     <joint name="chassis_joint" type="fixed">
       <origin xyz="${-tracker_base_offset_x} 0 0.193" rpy="0 0 0"/>
