Commit message: Fixed robot_state_publisher problems removed unecessary files changed base model for simulation

File: install/taurob_tracker_simulation/taurob_tracker_description/urdf/VLP-16.urdf.xacro (robot description, xacro)
@@ -18,10 +18,10 @@
       <visual>
         <geometry>
-          <mesh filename="package://taurob_tracker_description_sim/meshes/VLP16_base_1.dae" />
+          <mesh filename="package://taurob_tracker_description/meshes/VLP16_base_1.dae" />
         </geometry>
       </visual>
       <visual>
         <geometry>
-          <mesh filename="package://taurob_tracker_description_sim/meshes/VLP16_base_2.dae" />
+          <mesh filename="package://taurob_tracker_description/meshes/VLP16_base_2.dae" />
         </geometry>
       </visual>
@@ -47,5 +47,5 @@
         <origin xyz="0 0 -0.0377" />
         <geometry>
-          <mesh filename="package://taurob_tracker_description_sim/meshes/VLP16_scan.dae" />
+          <mesh filename="package://taurob_tracker_description/meshes/VLP16_scan.dae" />
         </geometry>
       </visual>
