Commit message: Fixed back camera error

File: install/taurob_tracker_simulation/taurob_tracker_description/urdf/taurob_tracker_flipper.xacro (robot description, xacro)
@@ -180,5 +180,5 @@
   <xacro:taurob_camera_gazebo link_name="camera_link_front" camera_name="camera_front" rtsp_support="false" />
   <xacro:taurob_camera suffix="back" parent="chassis_link">
-    <origin xyz="-0.6 0.0 ${-tracker_base_size_z*0.5}" rpy="0 0 0" />
+    <origin xyz="-0.6 0.0 ${-tracker_base_size_z*0.5}" rpy="0 0 ${M_PI}" />
   </xacro:taurob_camera>
   <xacro:taurob_camera_gazebo link_name="camera_link_back" camera_name="camera_back" rtsp_support="false"/>

Commit message: Fixed back camera

File: install/taurob_tracker_simulation/taurob_tracker_description/urdf/taurob_tracker_flipper.xacro (robot description, xacro)
@@ -184,5 +184,5 @@
   <xacro:taurob_camera_gazebo link_name="camera_link_back" camera_name="camera_back" rtsp_support="false"/>
   <xacro:taurob_camera suffix="elevated" parent="camera_mount">
-    <origin xyz="0 0 0" rpy="0 0 0" />
+    <origin xyz="0 0 0" rpy="0 0 ${M_PI}" />
   </xacro:taurob_camera>
   <xacro:taurob_camera_gazebo link_name="camera_link_elevated" camera_name="camera_elevated" rtsp_support="false"/>
